Commit message: body orientation joints

File: phantomx_description/urdf/phantomx.urdf (robot description, URDF)
Before this commit: robot PhantomX, 26 links, 25 joints
Links:
- added link base_rx
- added link base_ry
Joints:
- removed joint j_phantomx_attachment
- added joint j_body_rx: type continuous, parent base_link, child base_rx, origin xyz=0 0 0 rpy=0 0 0, axis 1 0 0
- added joint j_body_ry: type continuous, parent base_rx, child base_ry, origin xyz=0 0 0 rpy=0 0 0, axis 0 1 0
- added joint j_body_rz: type continuous, parent base_ry, child MP_BODY, origin xyz=0 0 0 rpy=0 0 0, axis 0 0 1

Commit message: Kinematic Chain and Jacobian

File: phantomx_description/urdf/phantomx.urdf (robot description, URDF)
Before this commit: robot PhantomX, 28 links, 27 joints
Links:
- removed link base_rx
- removed link base_ry
Joints:
- removed joint j_body_rx
- removed joint j_body_ry
- removed joint j_body_rz
- added joint j_phantomx_attachment: type fixed, parent base_link, child MP_BODY, origin xyz=0 0 0 rpy=0 0 0
